Commit message: 31

File: ros2_2_ws/src/my_robot_description/urdf/my_robot.urdf.xacro (robot description, xacro)
@@ -1,4 +1,10 @@
 <?xml version="1.0"?>
-<robot name="my_robot">
+<robot name="my_robot" xmlns:xacro="https://www.ros.org/wiki/xacro">
+    <!-- Xacro Variables-->
+    <xacro:property name="base_length" value="0.6" />
+    <xacro:property name="base_width" value="0.4" />
+    <xacro:property name="base_height" value="0.2" />
+    <xacro:property name="wheel_radius" value="0.1" />
+    <xacro:property name="wheel_length" value="0.05" />
     <!-- Green material -->
     <material name="green">
@@ -18,7 +24,7 @@
     <link name="base_link">
         <visual>
-            <origin xyz="0 0 0.1" rpy="0 0 0" />
+            <origin xyz="0 0 ${base_height/2}" rpy="0 0 0" />
             <geometry>
-                <box size="0.6 0.4 0.2" />
+                <box size="${base_length} ${base_width} ${base_height}" />
             </geometry>
             <material name="blue" />
@@ -29,21 +35,21 @@
         <parent link="footprint_link"/>
         <child link="base_link"/>
-        <origin xyz="0.0 0.0 0.1" rpy="0.0 0.0 0.0"/>
+        <origin xyz="0.0 0.0 ${wheel_radius}" rpy="0.0 0.0 0.0"/>
     </joint>
     <!-- Right wheel link-->
     <link name="right_wheel_link">
         <visual>
-            <origin xyz="0.0 0.0 0.0" rpy="1.57 0.0 0.0"/>
+            <origin xyz="0.0 0.0 0.0" rpy="${pi/2.0} 0.0 0.0"/>
             <geometry>
-                <cylinder radius="0.1" length="0.05"/>
+                <cylinder radius="${wheel_radius}" length="${wheel_length}"/>
             </geometry>
             <material name="grey" />
         </visual>
     </link>
-    <!-- Base right_Wheel joint -->
+    <!-- Base right_wheel joint -->
     <joint name="base_rightwheel_joint" type="continuous">
         <parent link="base_link"/>
         <child link="right_wheel_link"/>
-        <origin xyz="-0.15 -0.225 0.0" rpy="0.0 0.0 0.0"/>
+        <origin xyz="${-base_length/4.0} ${-base_width/2 - wheel_length/2} 0.0" rpy="0.0 0.0 0.0"/>
         <axis xyz="0.0 1.0 0.0"/>
     </joint>
@@ -51,5 +57,5 @@
     <link name="left_wheel_link">
         <visual>
-            <origin xyz="0.0 0.0 0.0" rpy="1.57 0.0 0.0"/>
+            <origin xyz="0.0 0.0 0.0" rpy="${pi/2.0} 0.0 0.0"/>
             <geometry>
                 <cylinder radius="0.1" length="0.05"/>
@@ -62,5 +68,5 @@
         <parent link="base_link"/>
         <child link="left_wheel_link"/>
-        <origin xyz="-0.15 0.225 0.0" rpy="0.0 0.0 0.0"/>
+        <origin xyz="${-base_length/4.0} ${base_width/2 + wheel_length/2} 0.0" rpy="0.0 0.0 0.0"/>
         <axis xyz="0.0 1.0 0.0"/>
     </joint>
@@ -70,5 +76,5 @@
             <origin xyz="0.0 0.0 0.0" rpy="0.0 0.0 0.0"/>
             <geometry>
-                <sphere radius="0.05"/>
+                <sphere radius="${wheel_radius/2}"/>
             </geometry>
             <material name="grey" />
@@ -79,5 +85,5 @@
         <parent link="base_link"/>
         <child link="caster_wheel_link"/>
-        <origin xyz="0.15 0.0 -0.05" rpy="0.0 0.0 0.0"/>
+        <origin xyz="${base_length/3.0} 0.0 ${-wheel_radius/2}" rpy="0.0 0.0 0.0"/>
     </joint>
 </robot>

Commit message: 32

File: ros2_2_ws/src/my_robot_description/urdf/my_robot.urdf.xacro (robot description, xacro)
@@ -3,7 +3,7 @@
     <!-- Xacro Variables-->
     <xacro:property name="base_length" value="0.6" />
-    <xacro:property name="base_width" value="0.4" />
-    <xacro:property name="base_height" value="0.2" />
-    <xacro:property name="wheel_radius" value="0.1" />
+    <xacro:property name="base_width" value="1.2" />
+    <xacro:property name="base_height" value="0.5" />
+    <xacro:property name="wheel_radius" value="0.5" />
     <xacro:property name="wheel_length" value="0.05" />
     <!-- Green material -->
@@ -59,5 +59,5 @@
             <origin xyz="0.0 0.0 0.0" rpy="${pi/2.0} 0.0 0.0"/>
             <geometry>
-                <cylinder radius="0.1" length="0.05"/>
+                <cylinder radius="${wheel_radius}" length="${wheel_length}"/>
             </geometry>
             <material name="grey" />

Commit message: 32

File: ros2_2_ws/src/my_robot_description/urdf/my_robot.urdf.xacro (robot description, xacro)
@@ -37,14 +37,18 @@
         <origin xyz="0.0 0.0 ${wheel_radius}" rpy="0.0 0.0 0.0"/>
     </joint>
+    <!-- wheel macro, predefined objects, just like in kivy-->
+    <xacro:macro name="wheel_link" params="prefix">
+        <link name="${prefix}_wheel_link">
+            <visual>
+                <origin xyz="0.0 0.0 0.0" rpy="${pi/2.0} 0.0 0.0"/>
+                <geometry>
+                    <cylinder radius="${wheel_radius}" length="${wheel_length}"/>
+                </geometry>
+                <material name="grey" />
+            </visual>
+        </link>
+    </xacro:macro>
     <!-- Right wheel link-->
-    <link name="right_wheel_link">
-        <visual>
-            <origin xyz="0.0 0.0 0.0" rpy="${pi/2.0} 0.0 0.0"/>
-            <geometry>
-                <cylinder radius="${wheel_radius}" length="${wheel_length}"/>
-            </geometry>
-            <material name="grey" />
-        </visual>
-    </link>
+    <xacro:wheel_link prefix="right" />
     <!-- Base right_wheel joint -->
     <joint name="base_rightwheel_joint" type="continuous">
@@ -55,13 +59,5 @@
     </joint>
     <!-- Left wheel link-->
-    <link name="left_wheel_link">
-        <visual>
-            <origin xyz="0.0 0.0 0.0" rpy="${pi/2.0} 0.0 0.0"/>
-            <geometry>
-                <cylinder radius="${wheel_radius}" length="${wheel_length}"/>
-            </geometry>
-            <material name="grey" />
-        </visual>
-    </link>
+    <xacro:wheel_link prefix="left" />
     <!-- Base left joint -->
     <joint name="base_leftwheel_joint" type="continuous">

Commit message: importing xacro into xacro

File: ros2_2_ws/src/my_robot_description/urdf/my_robot.urdf.xacro (robot description, xacro)
@@ -1,85 +1,6 @@
 <?xml version="1.0"?>
 <robot name="my_robot" xmlns:xacro="https://www.ros.org/wiki/xacro">
-    <!-- Xacro Variables-->
-    <xacro:property name="base_length" value="0.6" />
-    <xacro:property name="base_width" value="1.2" />
-    <xacro:property name="base_height" value="0.5" />
-    <xacro:property name="wheel_radius" value="0.5" />
-    <xacro:property name="wheel_length" value="0.05" />
-    <!-- Green material -->
-    <material name="green">
-        <color rgba="0 0.5 0 1"/>
-    </material>
-    <!-- Blue material -->
-    <material name="blue">
-        <color rgba="0 0 0.5 1"/>
-    </material>
-    <!-- Grey color-->
-    <material name="grey">
-        <color rgba="0.5 0.5 0.5 1"/>
-    </material>
-    <!-- base_footprint-->
-    <link name="footprint_link" />
-    <!-- Base link-->
-    <link name="base_link">
-        <visual>
-            <origin xyz="0 0 ${base_height/2}" rpy="0 0 0" />
-            <geometry>
-                <box size="${base_length} ${base_width} ${base_height}" />
-            </geometry>
-            <material name="blue" />
-        </visual>
-    </link>
-    <!-- footprint base joint-->
-    <joint name="footprint_base_joint" type="fixed">
-        <parent link="footprint_link"/>
-        <child link="base_link"/>
-        <origin xyz="0.0 0.0 ${wheel_radius}" rpy="0.0 0.0 0.0"/>
-    </joint>
-    <!-- wheel macro, predefined objects, just like in kivy-->
-    <xacro:macro name="wheel_link" params="prefix">
-        <link name="${prefix}_wheel_link">
-            <visual>
-                <origin xyz="0.0 0.0 0.0" rpy="${pi/2.0} 0.0 0.0"/>
-                <geometry>
-                    <cylinder radius="${wheel_radius}" length="${wheel_length}"/>
-                </geometry>
-                <material name="grey" />
-            </visual>
-        </link>
-    </xacro:macro>
-    <!-- Right wheel link-->
-    <xacro:wheel_link prefix="right" />
-    <!-- Base right_wheel joint -->
-    <joint name="base_rightwheel_joint" type="continuous">
-        <parent link="base_link"/>
-        <child link="right_wheel_link"/>
-        <origin xyz="${-base_length/4.0} ${-base_width/2 - wheel_length/2} 0.0" rpy="0.0 0.0 0.0"/>
-        <axis xyz="0.0 1.0 0.0"/>
-    </joint>
-    <!-- Left wheel link-->
-    <xacro:wheel_link prefix="left" />
-    <!-- Base left joint -->
-    <joint name="base_leftwheel_joint" type="continuous">
-        <parent link="base_link"/>
-        <child link="left_wheel_link"/>
-        <origin xyz="${-base_length/4.0} ${base_width/2 + wheel_length/2} 0.0" rpy="0.0 0.0 0.0"/>
-        <axis xyz="0.0 1.0 0.0"/>
-    </joint>
-    <!-- Caster wheel link-->
-    <link name="caster_wheel_link">
-        <visual>
-            <origin xyz="0.0 0.0 0.0" rpy="0.0 0.0 0.0"/>
-            <geometry>
-                <sphere radius="${wheel_radius/2}"/>
-            </geometry>
-            <material name="grey" />
-        </visual>
-    </link>
-    <!-- Casterwheel base joint-->
-    <joint name="caster_wheel_base_joint" type="fixed">
-        <parent link="base_link"/>
-        <child link="caster_wheel_link"/>
-        <origin xyz="${base_length/3.0} 0.0 ${-wheel_radius/2}" rpy="0.0 0.0 0.0"/>
-    </joint>
+    <!-- Xacro imports-->
+    <xacro:include filename="common_properties.xacro"/>
+    <xacro:include filename="mobile_base.xacro"/>
 </robot>
