Commit message: 44

File: ros2_2_ws/src/my_robot_description/urdf/mobile_base.xacro (robot description, xacro)
@@ -3,7 +3,7 @@
     <!-- Xacro Variables-->
     <xacro:property name="base_length" value="0.6" />
-    <xacro:property name="base_width" value="1.2" />
-    <xacro:property name="base_height" value="0.5" />
-    <xacro:property name="wheel_radius" value="0.5" />
+    <xacro:property name="base_width" value="0.4" />
+    <xacro:property name="base_height" value="0.2" />
+    <xacro:property name="wheel_radius" value="0.1" />
     <xacro:property name="wheel_length" value="0.05" />
     <!-- base_footprint-->
@@ -18,4 +18,10 @@
             <material name="blue" />
         </visual>
+        <collision>
+            <origin xyz="0 0 ${base_height/2}" rpy="0 0 0" />
+            <geometry>
+                <box size="${base_length} ${base_width} ${base_height}" />
+            </geometry>
+        </collision>
         <xacro:box_inertia m="5.0"
                            x="${base_length}" y="${base_width}" z="${base_height}"
@@ -38,4 +44,10 @@
                 <material name="grey" />
             </visual>
+            <collision>
+                <origin xyz="0.0 0.0 0.0" rpy="${pi/2.0} 0.0 0.0"/>
+                <geometry>
+                    <sphere radius="${wheel_radius}"/>
+                </geometry>
+            </collision>
             <xacro:cylinder_inertia m="1.0" r="${wheel_radius}" h="${wheel_length}"
                                     o_xyz="0 0 0" o_rpy="${pi/2} 0 0"/>
@@ -69,4 +81,10 @@
             <material name="grey" />
         </visual>
+        <collision>
+            <origin xyz="0.0 0.0 0.0" rpy="0.0 0.0 0.0"/>
+            <geometry>
+                <sphere radius="${wheel_radius/2}"/>
+            </geometry>
+        </collision>
         <xacro:sphere_inertia m="0.5" r="${wheel_radius/2}"
                                o_xyz="0 0 0" o_rpy="0 0 0"/>
