Commit message: 42

File: ros2_2_ws/src/my_robot_description/urdf/common_properties.xacro (robot description, xacro)
@@ -13,3 +13,33 @@
         <color rgba="0.5 0.5 0.5 1"/>
     </material>
+    <!-- Box Intertial macro-->
+    <xacro:macro name="box_inertia" params="m x y z o_xyz o_rpy">
+        <inertial>
+            <mass value="${m}" />
+            <origin xyz="${o_xyz}" rpy="${o_rpy}"/>
+            <inertia ixx="${(m/12) *(y*y + z*z)}" ixy="0" ixz="0"
+                     iyy="${(m/12)*(x*x + z*z)}" iyz="0"
+                     izz="${(m/12)*(y*y + x*x)}"/>
+        </inertial>
+    </xacro:macro>
+    <!-- Cylinder Intertial macro-->
+    <xacro:macro name="cylinder_inertia" params="m r h o_xyz o_rpy">
+        <inertial>
+            <mass value="${m}" />
+            <origin xyz="${o_xyz}" rpy="${o_rpy}"/>
+            <inertia ixx="${(m/12) *(3*r**2 + h**2)}" ixy="0" ixz="0"
+                     iyy="${(m/12) *(3*r**2 + h**2)}" iyz="0"
+                     izz="${(m*r**2)/2}"/>
+        </inertial>
+    </xacro:macro>
+    <!-- Sphere Intertial macro-->
+    <xacro:macro name="sphere_inertia" params="m r o_xyz o_rpy">
+        <inertial>
+            <mass value="${m}" />
+            <origin xyz="${o_xyz}" rpy="${o_rpy}"/>
+            <inertia ixx="${2*(m*r**2)/5}" ixy="0" ixz="0"
+                     iyy="${2*(m*r**2)/5}" iyz="0"
+                     izz="${2*(m*r**2)/5}"/>
+        </inertial>
+    </xacro:macro>
 </robot>

File: ros2_2_ws/src/my_robot_description/urdf/mobile_base.xacro (robot description, xacro)
@@ -18,4 +18,7 @@
             <material name="blue" />
         </visual>
+        <xacro:box_inertia m="5.0"
+                           x="${base_length}" y="${base_width}" z="${base_height}"
+                           o_xyz="0 0 ${base_height/2}" o_rpy="0 0 0" />
     </link>
     <!-- footprint base joint-->
@@ -35,4 +38,6 @@
                 <material name="grey" />
             </visual>
+            <xacro:cylinder_inertia m="1.0" r="${wheel_radius}" h="${wheel_length}"
+                                    o_xyz="0 0 0" o_rpy="${pi/2} 0 0"/>
         </link>
     </xacro:macro>
@@ -64,4 +69,6 @@
             <material name="grey" />
         </visual>
+        <xacro:sphere_inertia m="0.5" r="${wheel_radius/2}"
+                               o_xyz="0 0 0" o_rpy="0 0 0"/>
     </link>
     <!-- Casterwheel base joint-->

Commit message: complete robot with arm

File: ros2_2_ws/src/my_robot_description/urdf/common_properties.xacro (robot description, xacro)
@@ -12,4 +12,12 @@
     <material name="grey">
         <color rgba="0.5 0.5 0.5 1"/>
+    </material>
+    <!-- Yellow material -->
+    <material name="yellow">
+        <color rgba="1 1 0 1"/>
+    </material>
+    <!-- Orange material -->
+    <material name="orange">
+        <color rgba="1.0 0.647 0.0 1.0"/>
     </material>
     <!-- Box Intertial macro-->

File: ros2_2_ws/src/my_robot_description/urdf/my_robot.urdf.xacro (robot description, xacro)
@@ -6,3 +6,11 @@
     <xacro:include filename="mobile_base_gazebo.xacro"/>
     <xacro:include filename="camera.xacro"/>
+    <!-- Arm module -->
+    <xacro:include filename="arm_gazebo.xacro"/>
+    <xacro:include filename="arm.xacro"/>
+    <joint name="car_arm_joint" type="fixed">
+        <parent link="base_link"/>
+        <child link="arm_base_link"/>
+        <origin xyz="${base_length/4} 0.0 ${base_height}" rpy="0.0 0.0 ${pi/2}"/>
+    </joint>
 </robot>
