Commit message: second course

File: ros2_2_ws/src/my_robot_description/urdf/arm.xacro (robot description, xacro)
@@ -5,5 +5,5 @@
     <xacro:property name="box_width" value="0.1" />
     <xacro:property name="box_height" value="0.02" />
-    <xacro:property name="box_mass" value="5"/>
+    <xacro:property name="box_mass" value="0.5"/>
     <xacro:property name="forearm_radius" value="0.02"/>
     <xacro:property name="forearm_length" value="0.3"/>
